Commit message: 增加了gitignore

File: src/fr5_description/urdf/fr5_description.gazebo.xacro (robot description, xacro)
@@ -13,5 +13,25 @@
     <plugin name="gazebo_ros_control" filename="libgazebo_ros_control.so">
       <robotNamespace>/</robotNamespace>
+      <robotSimType>gazebo_ros_control/DefaultRobotHWSim</robotSimType>
     </plugin>
+  </gazebo>
+  <!-- Gazebo properties for each joint to improve stability -->
+  <gazebo reference="j1">
+    <implicitSpringDamper>true</implicitSpringDamper>
+  </gazebo>
+  <gazebo reference="j2">
+    <implicitSpringDamper>true</implicitSpringDamper>
+  </gazebo>
+  <gazebo reference="j3">
+    <implicitSpringDamper>true</implicitSpringDamper>
+  </gazebo>
+  <gazebo reference="j4">
+    <implicitSpringDamper>true</implicitSpringDamper>
+  </gazebo>
+  <gazebo reference="j5">
+    <implicitSpringDamper>true</implicitSpringDamper>
+  </gazebo>
+  <gazebo reference="j6">
+    <implicitSpringDamper>true</implicitSpringDamper>
   </gazebo>
   <!-- Transmission for joint 1 -->

File: src/fr5_description/urdf/fr5_description.urdf (robot description, URDF)
Before this commit: robot fr5_description, 7 links, 6 joints
Joints:
- joint j5: limit lower=0 upper=6.1958 effort=500 velocity=3.14 -> lower=0 upper=6.2832 effort=500 velocity=3.14
